File: Integrated-SC-system/Active_Balancing.sch (KiCad schematic (older format))
At the start: 7 parts, among them IC1 ALD910017SALI

Commit message: Update
Other:
- note added: "160ohm"
- note added: "Removed from prototype"
Changed lines of the file:
@@
 $Descr A4 11693 8268
 encoding utf-8
-Sheet 7 27
+Sheet 4 27
 Title ""
 Date ""
@@
 AR Path="/601B19F6/601286E7" Ref="IC5"  Part="1"
 AR Path="/601B304B/601286E7" Ref="IC6"  Part="1"
-F 0 "IC6" H 4650 2915 50  0000 C CNN
+F 0 "IC3" H 4650 2915 50  0000 C CNN
 F 1 "ALD910017SALI" H 4650 2824 50  0000 C CNN
 F 2 "SamacSys_Parts:SOIC127P600X175-8N" H 5100 2750 50  0001 L CNN
@@
 AR Path="/601B19F6/6012F617" Ref="D10"  Part="1"
 AR Path="/601B304B/6012F617" Ref="D12"  Part="1"
-F 0 "D12" H 6300 3165 50  0000 C CNN
+F 0 "D6" H 6300 3165 50  0000 C CNN
 F 1 "FSV10100V" H 6300 3074 50  0000 C CNN
 F 2 "SamacSys_Parts:FSV20100V" H 6600 3000 50  0001 L CNN
@@
 AR Path="/601B19F6/6051A426" Ref="R17"  Part="1"
 AR Path="/601B304B/6051A426" Ref="R21"  Part="1"
-F 0 "R21" H 6520 2296 50  0000 L CNN
+F 0 "R9" H 6520 2296 50  0000 L CNN
 F 1 "400" H 6520 2205 50  0000 L CNN
 F 2 "Resistor_SMD:R_1206_3216Metric_Pad1.30x1.75mm_HandSolder" V 6380 2250 50  0001 C CNN
@@
 AR Path="/601B19F6/6051A8EE" Ref="R18"  Part="1"
 AR Path="/601B304B/6051A8EE" Ref="R22"  Part="1"
-F 0 "R22" H 6520 2696 50  0000 L CNN
+F 0 "R10" H 6520 2696 50  0000 L CNN
 F 1 "400" H 6520 2605 50  0000 L CNN
 F 2 "Resistor_SMD:R_1206_3216Metric_Pad1.30x1.75mm_HandSolder" V 6380 2650 50  0001 C CNN
@@
 AR Path="/601B19F6/6051C010" Ref="R19"  Part="1"
 AR Path="/601B304B/6051C010" Ref="R23"  Part="1"
-F 0 "R23" H 6520 3196 50  0000 L CNN
+F 0 "R11" H 6520 3196 50  0000 L CNN
 F 1 "400" H 6520 3105 50  0000 L CNN
 F 2 "Resistor_SMD:R_1206_3216Metric_Pad1.30x1.75mm_HandSolder" V 6380 3150 50  0001 C CNN
@@
 AR Path="/601B19F6/6051C018" Ref="R20"  Part="1"
 AR Path="/601B304B/6051C018" Ref="R24"  Part="1"
-F 0 "R24" H 6520 3596 50  0000 L CNN
+F 0 "R12" H 6520 3596 50  0000 L CNN
 F 1 "400" H 6520 3505 50  0000 L CNN
 F 2 "Resistor_SMD:R_1206_3216Metric_Pad1.30x1.75mm_HandSolder" V 6380 3550 50  0001 C CNN
@@
 AR Path="/601B19F6/6012650E" Ref="D9"  Part="1"
 AR Path="/601B304B/6012650E" Ref="D11"  Part="1"
-F 0 "D11" H 6300 2265 50  0000 C CNN
+F 0 "D5" H 6300 2265 50  0000 C CNN
 F 1 "FSV10100V" H 6300 2174 50  0000 C CNN
 F 2 "SamacSys_Parts:FSV20100V" H 6600 2100 50  0001 L CNN
@@
 	0    1    1    0
 $EndComp
+Wire Notes Line
+	5500 2500 5500 1950
+Wire Notes Line
+	5500 1950 6150 1950
+Wire Notes Line
+	6150 1950 6150 3950
+Wire Notes Line
+	6150 3950 5350 3950
+Wire Notes Line
+	5350 3950 5350 3300
+Wire Notes Line
+	5350 3300 4000 3300
+Wire Notes Line
+	4000 3300 4000 2500
+Wire Notes Line
+	4000 2500 5500 2500
+Text Notes 4300 3450 0    50   ~ 0
+Removed from prototype
+Text Notes 6700 2450 0    50   ~ 0
+160ohm
+Text Notes 6700 3400 0    50   ~ 0
+160ohm
 $EndSCHEMATC
