File: Integrated-SC-system/Overvoltage_Protection.sch (KiCad schematic (older format))
At the start: 14 parts, among them IC10 OPA197IDR, IC31 BD4827G-TR

Commit message: Update
Other:
- note added: "47kOhm"
